File: LogicGateDisplaySolder.kicad_pcb (KiCad board)
At the start: 2 copper layers, 100 x 100 mm, 37 parts, among them Q3 NPN, Q4 NPN, Q5 NPN, Q6 NPN, Q7 NPN, Q8 NPN, SW1 SW_Push, SW2 SW_Push, SW3 SW_Push, SW4 SW_Push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

Commit message: update
Parts:
- removed C1: C, Capacitor_THT:CP_Radial_D8.0mm_P5.00mm
Connections:
- BT1 pad 2: Net-(BT1--) -> ground
Routing:
- net ground: track 478.2 -> 499.5 mm
- net Net-(BT1--): track 19.9 -> 0.00 mm
Other:
- outline, holes or cut-outs redrawn
